Commit message: Refine locomotion training setup

File: assets/source/bello/full_body/urdf/bello_full_body.urdf (robot description, URDF)
Before this commit: robot bello_full_body, 45 links, 44 joints
Links:
- link left_ankle_roll_link: geometry collision box size=0.026 0.04 0.05; collision box size=0.106 0.17007 0.05
- link right_ankle_roll_link: geometry collision box size=0.026 0.04 0.05; collision box size=0.106 0.17007 0.05

File: assets/source/bello/lower_body/urdf/bello_lower_body.urdf (robot description, URDF)
Before this commit: robot bello_leg_urdf, 13 links, 12 joints
Links:
- link left_ankle_roll_link: geometry collision box size=0.026 0.04 0.05; collision box size=0.106 0.17007 0.05
- link right_ankle_roll_link: geometry collision box size=0.026 0.04 0.05; collision box size=0.106 0.17007 0.05

Commit message: Add fifth foot collision primitive

File: assets/source/bello/full_body/urdf/bello_full_body.urdf (robot description, URDF)
Before this commit: robot bello_full_body, 45 links, 44 joints
Links:
- link left_ankle_roll_link: geometry collision box size=0.026 0.04 0.05; collision box size=0.106 0.04195 0.05
- link right_ankle_roll_link: geometry collision box size=0.026 0.04 0.05; collision box size=0.106 0.04195 0.05

File: assets/source/bello/lower_body/urdf/bello_lower_body.urdf (robot description, URDF)
Before this commit: robot bello_leg_urdf, 13 links, 12 joints
Links:
- link left_ankle_roll_link: geometry collision box size=0.026 0.04 0.05; collision box size=0.106 0.04195 0.05
- link right_ankle_roll_link: geometry collision box size=0.026 0.04 0.05; collision box size=0.106 0.04195 0.05
